File: KiCad Schemantics/d_latch_bb_t_1/d_latch_bb_t_1.kicad_sch (KiCad schematic)
At the start: 10 parts

Commit message: Optimized the D Latch Test
Parts:
- removed D?: LED, symbol Device:LED
- removed D?: (no value), symbol Device:LED
- removed R? (x3): (no value), symbol Device:R
- removed R?: 220 Ohm, symbol Device:R
- removed SW?: SW_Push, symbol Switch:SW_Push
- removed SW?: (no value), symbol Switch:SW_Push
- removed U?: (no value), symbol Gosheto:74LS02_(NOR)
- removed U?: (no value), symbol Gosheto:74LS08_(AND)
- added D? (x2): LED, symbol Device:LED
- added R? (x4): 220 Ohm, symbol Device:R
- added SW? (x2): SW_Push, symbol Switch:SW_Push
- added U?: 74LS02_(NOR), symbol Gosheto:74LS02_(NOR)
- added U?: 74LS08_(AND), symbol Gosheto:74LS08_(AND)
Connections:
- net +: now also SW?.2, SW?.2
- net -: now also R?.1, R?.1, R?.2, R?.2
- new net: D?.1 (K), R?.1 (x2)
- new net: R?.2, SW?.1 (x2)
Other:
- note added: "Inverting the D's output through NOR gate"
- note added: "O_{1}"
- note added: "O_{2}"
- note added: "enable_switcher тест"
- note added: "~{D}"

Commit message: Notes for the enable switch schemantic
Other:
- note added: "Просто тествам как работи Enable-a. Eg: При натискане позволява стойноста на D да вземе ефект."
Changed lines of the file:
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@@
     (effects (font (size 0.6 0.6)) (justify left bottom))
+  )
+  (text "Просто тествам как работи Enable-a. Eg: При \nнатискане позволява стойноста на D да вземе ефект."
+    (at 123.19 58.42 0)
+    (effects (font (size 0.8 0.8)) (justify left bottom))
   )
   (text "D" (at 117.094 82.804 0)
